File: KiCAD_files/business_card/business_card.kicad_pcb (KiCad board)
At the start: 2 copper layers, 88.9 x 50.8 mm, 200 parts, among them J2 Conn_01x05_Pin, Q1 AO3401A, SW1 CS1210F260, SW2 CS1210F260, SW3 CS1210F260, U1 STM32U073CCUx, U2 ST25DV04KC-IE6S3

Commit message: Initial Layout for V2.0
Parts:
- removed the D1 at (114.6, 68.1)
- removed the D1 at (93.2, 64.5)
- removed the D1 at (111.0, 82.3)
- removed the D1 at (111.0, 78.7)
- removed the D1 at (96.7, 78.7)
- removed the D1 at (103.9, 78.7)
- removed the D1 at (93.2, 82.3)
- removed the D1 at (103.9, 71.6)
- removed the D1 at (96.7, 64.5)
- removed the D1 at (107.4, 75.2)
- removed the D1 at (93.2, 75.2)
- removed the D1 at (93.2, 68.1)
- removed the D1 at (93.2, 78.7)
- removed the D1 at (103.9, 82.3)
- removed the D1 at (103.9, 68.1)
- removed the D1 at (100.3, 82.3)
- removed the D1 at (111.0, 71.6)
- removed the D1 at (100.3, 68.1)
- removed the D1 at (96.7, 68.1)
- removed the D1 at (107.4, 71.6)
- removed the D1 at (111.0, 75.2)
- removed the D1 at (107.4, 68.1)
- removed the D1 at (114.6, 71.6)
- removed the D1 at (93.2, 71.6)
- removed the D1 at (96.7, 71.6)
- removed the D1 at (114.6, 64.5)
- removed the D1 at (100.3, 71.6)
- removed the D1 at (107.4, 82.3)
- removed the D1 at (100.3, 64.5)
- removed the D1 at (96.7, 75.2)
- removed the D1 at (96.7, 82.3)
- removed the D1 at (114.6, 78.7)
- removed the D1 at (100.3, 78.7)
- removed the D1 at (107.4, 78.7)
- removed the D1 at (100.3, 75.2)
- removed the D1 at (114.6, 75.2)
- removed the D1 at (103.9, 75.2)
- removed the D1 at (107.4, 64.5)
- removed the D1 at (111.0, 68.1)
- removed the D1 at (103.9, 64.5)
- removed the D1 at (114.6, 82.3)
- removed the D1 at (111.0, 64.5)
- removed the D2 at (96.7, 72.9)
- removed the D2 at (107.4, 65.8)
- removed the D2 at (93.2, 65.8)
- removed the D2 at (100.3, 76.5)
- removed the D2 at (111.0, 83.6)
- removed the D2 at (107.4, 76.5)
- removed the D2 at (111.0, 72.9)
- removed the D2 at (93.2, 72.9)
- removed the D2 at (114.6, 72.9)
- removed the D2 at (103.9, 76.5)
- removed the D2 at (107.4, 72.9)
- removed the D2 at (103.9, 65.8)
- removed the D2 at (107.4, 69.3)
- removed the D2 at (100.3, 80.0)
- removed the D2 at (96.7, 80.0)
- removed the D2 at (114.6, 69.3)
- removed the D2 at (93.2, 76.5)
- removed the D2 at (103.9, 69.3)
- removed the D2 at (114.6, 83.6)
- removed the D2 at (107.4, 80.0)
- removed the D2 at (114.6, 65.8)
- removed the D2 at (100.3, 65.8)
- removed the D2 at (103.9, 72.9)
- removed the D2 at (93.2, 83.6)
- removed the D2 at (103.9, 83.6)
- removed the D2 at (96.7, 69.3)
- removed the D2 at (114.6, 80.0)
- removed the D2 at (100.3, 72.9)
- removed the D2 at (93.2, 80.0)
- removed the D2 at (100.3, 69.3)
- removed the D2 at (96.7, 76.5)
- removed the D2 at (103.9, 80.0)
- removed the D2 at (111.0, 65.8)
- removed the D2 at (111.0, 80.0)
- removed the D2 at (111.0, 69.3)
- removed the D2 at (111.0, 76.5)
- removed the D2 at (114.6, 76.5)
- removed the D2 at (100.3, 83.6)
- removed the D2 at (93.2, 69.3)
- removed the D2 at (96.7, 83.6)
- removed the D2 at (96.7, 65.8)
- removed the D2 at (107.4, 83.6)
- removed TP1: VDD, TestPoint:TestPoint_THTPad_D1.0mm_Drill0.5mm
- removed TP2: GND, TestPoint:TestPoint_THTPad_D1.0mm_Drill0.5mm
- removed TP3: SDA, TestPoint:TestPoint_THTPad_D1.0mm_Drill0.5mm
- removed TP4: SCL, TestPoint:TestPoint_THTPad_D1.0mm_Drill0.5mm
- added D1: RED, custom_footprints:LED_0603_1608Metric, F.Cu at (93.4, 67.6)
- added D2: ORN, custom_footprints:LED_0603_1608Metric, F.Cu at (93.4, 68.7)
- D10, D11, D12, D13, D14, D15, D16, D17, D18, D19, D20, D21, D22, D23, D24, D25, D26, D27, D28, D29, D3, D30, D31, D32, D33, D34, D35, D36, D37, D38, D39, D4, D40, D41, D42, D43, D44, D45, D46, D47, D48, D49, D5, D50, D51, D52, D53, D54, D55, D56, D57, D58, D59, D6, D60, D61, D62, D63, D64, D65, D66, D67, D68, D69, D7, D70, D71, D72, D73, D74, D75, D76, D77, D78, D79, D8, D80, D81, D82, D83, D84, D9: footprint LED_SMD:LED_0603_1608Metric -> custom_footprints:LED_0603_1608Metric
- moved D13 64.3 mm to (112.6, 67.6)
- moved D12 60.1 mm to (109.3, 68.7), turned to 180 degrees
- moved D11 59.7 mm to (109.3, 67.5)
- moved D14 57.7 mm to (112.6, 68.7), turned to 180 degrees
- moved D26 56.0 mm to (109.3, 71.9), turned to 180 degrees
- moved D25 55.6 mm to (109.3, 70.7)
- moved D10 55.6 mm to (106.0, 68.6), turned to 180 degrees
- moved D9 55.3 mm to (106.0, 67.5)
- moved D27 54.2 mm to (112.6, 70.7)
- moved D28 53.9 mm to (112.6, 71.9), turned to 180 degrees
- moved D39 51.5 mm to (109.3, 73.9)
- moved D8 51.5 mm to (102.9, 68.6), turned to 180 degrees
- moved D24 51.5 mm to (106.1, 71.9), turned to 180 degrees
- moved D7 51.3 mm to (102.9, 67.5)
- moved D23 51.2 mm to (106.1, 70.7)
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Connections:
- D25 pad 1: unconnected-(D25-K-Pad1) -> /COL6
- J2 pad 1: VDD -> GND
- J2 pad 2: /SWDIO -> /NRST
- J2 pad 3: /NRST -> /SWCLK
- J2 pad 4: /SWCLK -> /SWDIO
- J2 pad 5: GND -> VDD
- SW1 pad 1: /INPUT_DOWN -> unconnected-(SW1-Pad1)
- SW1 pad 2: unconnected-(SW1-Pad2) -> /INPUT_DOWN
- SW1 pad 3: unconnected-(SW1-K-Pad3) -> VDD
- SW2 pad 1: /INPUT_LEFT -> unconnected-(SW2-Pad1)
- SW2 pad 2: unconnected-(SW2-Pad2) -> /INPUT_LEFT
- SW2 pad 3: unconnected-(SW2-K-Pad3) -> VDD
- SW2 pad 4: VDD -> unconnected-(SW2-A-Pad4)
- SW3 pad 1: /INPUT_RIGHT -> unconnected-(SW3-Pad1)
- SW3 pad 2: unconnected-(SW3-Pad2) -> /INPUT_RIGHT
- U1 pad 11: /INPUT_DOWN -> unconnected-(U1-PA1-Pad11)
- U1 pad 12: /INPUT_LEFT -> unconnected-(U1-PA2-Pad12)
- U1 pad 13: /INPUT_RIGHT -> unconnected-(U1-PA3-Pad13)
- U1 pad 18: /ROW6 -> /ROW1
- U1 pad 19: /ROW5 -> /ROW2
- U1 pad 20: /ROW4 -> /ROW3
- U1 pad 29: unconnected-(U1-PA8-Pad29) -> /INPUT_RIGHT
- U1 pad 30: unconnected-(U1-PA9-Pad30) -> /INPUT_LEFT
- U1 pad 31: unconnected-(U1-PA10-Pad31) -> /INPUT_DOWN
- U1 pad 39: /ROW3 -> /ROW4
- U1 pad 40: /ROW2 -> /ROW5
- U1 pad 41: /ROW1 -> /ROW6
- U1 pad 42: /COL1 -> /COL4
- U1 pad 43: /COL2 -> /COL3
- U1 pad 45: /COL3 -> /COL2
- U1 pad 46: /COL4 -> /COL1
Routing:
- net VDD: track 0.00 -> 126.5 mm, vias 0 -> 4
- net GND: track 0.00 -> 101.3 mm, vias 0 -> 16
- net /COL1: track 0.00 -> 63.0 mm
- net /COL2: track 0.00 -> 58.9 mm
- net /COL3: track 0.00 -> 53.7 mm
- net /COL4: track 0.00 -> 50.0 mm
- net /COL5: track 0.00 -> 38.2 mm, vias 0 -> 2
- net Net-(D1-A): track 0.00 -> 36.6 mm, vias 0 -> 7
- net /INPUT_LEFT: track 0.00 -> 36.4 mm, vias 0 -> 2
- net Net-(D29-A): track 0.00 -> 36.1 mm, vias 0 -> 7
- net Net-(D15-A): track 0.00 -> 36.1 mm, vias 0 -> 7
- net /NRST: track 0.00 -> 35.6 mm, vias 0 -> 1
- net Net-(D43-A): track 0.00 -> 35.4 mm, vias 0 -> 7
- net Net-(D57-A): track 0.00 -> 35.3 mm, vias 0 -> 7
- net Net-(D71-A): track 0.00 -> 35.1 mm, vias 0 -> 7
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