File: KiCAD_files/business_card/business_card.kicad_sch (KiCad schematic)
At the start: 113 parts, among them J2 Conn_01x05_Pin, Q1 AO3401A, SW1 CS1210F260, SW2 CS1210F260, SW3 CS1210F260, U1 STM32U073CCUx, U2 ST25TN01K-AFH5

Commit message: Change Debug Interface Connector Size
Parts:
- J2: footprint Connector_PinHeader_1.00mm:PinHeader_1x05_P1.00mm_Vertical -> Connector_PinHeader_2.54mm:PinHeader_1x05_P2.54mm_Vertical
Changed lines of the file:
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@@
 	(title_block
 		(title "Connect_4_Business_Card")
-		(date "2026-03-16")
-		(rev "0")
+		(date "2026-05-15")
+		(rev "1")
 	)
 	(rectangle
@@
 			)
 		)
-		(property "Footprint" "Connector_PinHeader_1.00mm:PinHeader_1x05_P1.00mm_Vertical"
+		(property "Footprint" "Connector_PinHeader_2.54mm:PinHeader_1x05_P2.54mm_Vertical"
 			(at 48.26 69.85 0)
 			(hide yes)
